Commit message: sdfasdf

File: drake-distro/drake/solvers/trajectoryOptimization/dev/cylinder1.urdf (robot description, URDF)
Before this commit: robot cylinder, 1 links, 0 joints
Links:
- link cylinder: mass 1.397598 -> 1.542700

File: drake-distro/drake/solvers/trajectoryOptimization/dev/cylinder2.urdf (robot description, URDF)
Before this commit: robot cylinder, 1 links, 0 joints
Links:
- link cylinder: mass 1.397598 -> 1.712400

Commit message: aSdfasdf

File: drake-distro/drake/solvers/trajectoryOptimization/dev/cylinder1.urdf (robot description, URDF)
Before this commit: robot cylinder, 1 links, 0 joints
Links:
- link cylinder: mass 1.542700 -> 1.138624

File: drake-distro/drake/solvers/trajectoryOptimization/dev/cylinder2.urdf (robot description, URDF)
Before this commit: robot cylinder, 1 links, 0 joints
Links:
- link cylinder: mass 1.712400 -> 1.929264

Commit message: Adding data

File: drake-distro/drake/solvers/trajectoryOptimization/dev/cylinder1.urdf (robot description, URDF)
Before this commit: robot cylinder, 1 links, 0 joints
Links:
- link cylinder: mass 1.138624 -> 2.000000; geometry collision cylinder length=0.153584 radius=0.006659; visual cylinder length=0.153584 radius=0.006659

File: drake-distro/drake/solvers/trajectoryOptimization/dev/cylinder2.urdf (robot description, URDF)
Before this commit: robot cylinder, 1 links, 0 joints
Links:
- link cylinder: mass 1.929264 -> 2.000000; geometry collision cylinder length=0.153584 radius=0.006659; visual cylinder length=0.153584 radius=0.006659

Commit message: COmmiting before doing new observations

File: drake-distro/drake/solvers/trajectoryOptimization/dev/cylinder1.urdf (robot description, URDF)
Before this commit: robot cylinder, 1 links, 0 joints
Links:
- link cylinder: mass 2.000000 -> 1.000000; geometry collision cylinder length=0.260716 radius=0.081361; visual cylinder length=0.260716 radius=0.081361

Commit message: ASDF

File: drake-distro/drake/solvers/trajectoryOptimization/dev/cylinder1.urdf (robot description, URDF)
Before this commit: robot cylinder, 1 links, 0 joints
Links:
- link cylinder: mass 1.000000 -> 2.000000; geometry collision cylinder length=0.153584 radius=0.006659; visual cylinder length=0.153584 radius=0.006659

Commit message: sdf

File: drake-distro/drake/solvers/trajectoryOptimization/dev/cylinder1.urdf (robot description, URDF)
Before this commit: robot cylinder, 1 links, 0 joints
Links:
- link cylinder: mass 2.000000 -> 1.000000; geometry collision cylinder length=0.194054 radius=0.054400; visual cylinder length=0.194054 radius=0.054400

File: drake-distro/drake/solvers/trajectoryOptimization/dev/cylinder2.urdf (robot description, URDF)
Before this commit: robot cylinder, 1 links, 0 joints
Links:
- link cylinder: geometry collision cylinder length=0.486608 radius=0.132393; visual cylinder length=0.486608 radius=0.132393

Commit message: SDFASDF

File: drake-distro/drake/solvers/trajectoryOptimization/dev/cylinder1.urdf (robot description, URDF)
Before this commit: robot cylinder, 1 links, 0 joints
Links:
- link cylinder: mass 1.000000 -> 2.000000; geometry collision cylinder length=0.490508 radius=0.042261; visual cylinder length=0.490508 radius=0.042261

File: drake-distro/drake/solvers/trajectoryOptimization/dev/cylinder2.urdf (robot description, URDF)
Before this commit: robot cylinder, 1 links, 0 joints
Links:
- link cylinder: geometry collision cylinder length=0.490508 radius=0.042261; visual cylinder length=0.490508 radius=0.042261

Commit message: isadf

File: drake-distro/drake/solvers/trajectoryOptimization/dev/cylinder1.urdf (robot description, URDF)
Before this commit: robot cylinder, 1 links, 0 joints
Links:
- link cylinder: geometry collision cylinder length=0.486608 radius=0.132393; visual cylinder length=0.486608 radius=0.132393

File: drake-distro/drake/solvers/trajectoryOptimization/dev/cylinder2.urdf (robot description, URDF)
Before this commit: robot cylinder, 1 links, 0 joints
Links:
- link cylinder: geometry collision cylinder length=0.486608 radius=0.132393; visual cylinder length=0.486608 radius=0.132393

Commit message: lets make plots

File: drake-distro/drake/solvers/trajectoryOptimization/dev/cylinder1.urdf (robot description, URDF)
Before this commit: robot cylinder, 1 links, 0 joints
Links:
- link cylinder: mass 2.000000 -> 1.000000; geometry collision cylinder length=0.319803 radius=0.064447; visual cylinder length=0.319803 radius=0.064447

File: drake-distro/drake/solvers/trajectoryOptimization/dev/cylinder2.urdf (robot description, URDF)
Before this commit: robot cylinder, 1 links, 0 joints
Links:
- link cylinder: geometry collision cylinder length=0.370307 radius=0.038584; visual cylinder length=0.370307 radius=0.038584

Commit message: asdf

File: drake-distro/drake/solvers/trajectoryOptimization/dev/cylinder1.urdf (robot description, URDF)
Before this commit: robot cylinder, 1 links, 0 joints
Links:
- link cylinder: mass 1.000000 -> 2.000000; geometry collision cylinder length=0.153584 radius=0.006659; visual cylinder length=0.153584 radius=0.006659

File: drake-distro/drake/solvers/trajectoryOptimization/dev/cylinder2.urdf (robot description, URDF)
Before this commit: robot cylinder, 1 links, 0 joints
Links:
- link cylinder: geometry collision cylinder length=0.153584 radius=0.006659; visual cylinder length=0.153584 radius=0.006659

Commit message: sadfsafd

File: drake-distro/drake/solvers/trajectoryOptimization/dev/cylinder1.urdf (robot description, URDF)
Before this commit: robot cylinder, 1 links, 0 joints
Links:
- link cylinder: geometry collision cylinder length=0.370307 radius=0.038584; visual cylinder length=0.370307 radius=0.038584

File: drake-distro/drake/solvers/trajectoryOptimization/dev/cylinder2.urdf (robot description, URDF)
Before this commit: robot cylinder, 1 links, 0 joints
Links:
- link cylinder: geometry collision cylinder length=0.370307 radius=0.038584; visual cylinder length=0.370307 radius=0.038584

Commit message: asdasd

File: drake-distro/drake/solvers/trajectoryOptimization/dev/cylinder1.urdf (robot description, URDF)
Before this commit: robot cylinder, 1 links, 0 joints
Links:
- link cylinder: geometry collision cylinder length=0.590606 radius=0.243888; visual cylinder length=0.590606 radius=0.243888

File: drake-distro/drake/solvers/trajectoryOptimization/dev/cylinder2.urdf (robot description, URDF)
Before this commit: robot cylinder, 1 links, 0 joints
Links:
- link cylinder: geometry collision cylinder length=0.590606 radius=0.243888; visual cylinder length=0.590606 radius=0.243888

Commit message: asdf

File: drake-distro/drake/solvers/trajectoryOptimization/dev/cylinder1.urdf (robot description, URDF)
Before this commit: robot cylinder, 1 links, 0 joints
Links:
- link cylinder: mass 2.000000 -> 1.000000; geometry collision cylinder length=0.328078 radius=0.181223; visual cylinder length=0.328078 radius=0.181223

File: drake-distro/drake/solvers/trajectoryOptimization/dev/cylinder2.urdf (robot description, URDF)
Before this commit: robot cylinder, 1 links, 0 joints
Links:
- link cylinder: geometry collision cylinder length=0.446081 radius=0.111354; visual cylinder length=0.446081 radius=0.111354
